File:  MPU6050_Gyroscope.kicad_sch (KiCad schematic)
At the start: 7 parts, among them U6 MPU-6050

Commit message: Add files via upload
Parts:
- C20, C? (x2): footprint (none) -> Capacitor_SMD:C_0603_1608Metric; MPN (none) -> CC0603KRX7R9BB104
- C21: footprint (none) -> Capacitor_SMD:C_0603_1608Metric; MPN (none) -> 0603B222K500NT
- C?: footprint (none) -> Capacitor_SMD:C_0603_1608Metric; MPN (none) -> CL10A106KP8NNNC
- C?: value 0.01uF -> 10nF; footprint (none) -> Capacitor_SMD:C_0603_1608Metric; MPN (none) -> 0603B103K500NT
- U6: MPN (none) -> MPU-6050
Changed lines of the file:
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@@
       (effects (font (size 1.27 1.27)) (justify left))
     )
-    (property "Footprint" "" (at 117.475 74.295 0)
+    (property "Footprint" "Capacitor_SMD:C_0603_1608Metric" (at 117.475 74.295 0)
       (effects (font (size 1.27 1.27)) hide)
     )
     (property "Datasheet" "~" (at 117.475 74.295 0)
+      (effects (font (size 1.27 1.27)) hide)
+    )
+    (property "MPN" "CC0603KRX7R9BB104" (at 117.475 74.295 0)
       (effects (font (size 1.27 1.27)) hide)
     )
@@
       (effects (font (size 1.27 1.27)) (justify left))
     )
-    (property "Footprint" "" (at 170.815 111.76 0)
+    (property "Footprint" "Capacitor_SMD:C_0603_1608Metric" (at 170.815 111.76 0)
       (effects (font (size 1.27 1.27)) hide)
     )
@@
       (effects (font (size 1.27 1.27)) hide)
     )
+    (property "MPN" "0603B222K500NT" (at 170.815 111.76 0)
+      (effects (font (size 1.27 1.27)) hide)
+    )
     (pin "1")
     (pin "2")
@@
       (effects (font (size 1.27 1.27)) (justify left))
     )
-    (property "Footprint" "" (at 112.395 74.295 0)
+    (property "Footprint" "Capacitor_SMD:C_0603_1608Metric" (at 112.395 74.295 0)
       (effects (font (size 1.27 1.27)) hide)
     )
@@
       (effects (font (size 1.27 1.27)) hide)
     )
+    (property "MPN" "CL10A106KP8NNNC" (at 112.395 74.295 0)
+      (effects (font (size 1.27 1.27)) hide)
+    )
     (pin "1")
     (pin "2")
@@
       (effects (font (size 1.27 1.27)) (justify left))
     )
-    (property "Value" "0.01uF" (at 133.985 75.565 0)
-      (effects (font (size 1.27 1.27)) (justify left))
-    )
-    (property "Footprint" "" (at 135.89 74.295 0)
+    (property "Value" "10nF" (at 133.985 75.565 0)
+      (effects (font (size 1.27 1.27)) (justify left))
+    )
+    (property "Footprint" "Capacitor_SMD:C_0603_1608Metric" (at 135.89 74.295 0)
       (effects (font (size 1.27 1.27)) hide)
     )
     (property "Datasheet" "~" (at 135.89 74.295 0)
+      (effects (font (size 1.27 1.27)) hide)
+    )
+    (property "MPN" "0603B103K500NT" (at 135.89 74.295 0)
       (effects (font (size 1.27 1.27)) hide)
     )
@@
       (effects (font (size 1.27 1.27)) (justify left))
     )
-    (property "Footprint" "" (at 158.75 111.76 0)
+    (property "Footprint" "Capacitor_SMD:C_0603_1608Metric" (at 158.75 111.76 0)
       (effects (font (size 1.27 1.27)) hide)
     )
@@
       (effects (font (size 1.27 1.27)) hide)
     )
+    (property "MPN" "CC0603KRX7R9BB104" (at 158.75 111.76 0)
+      (effects (font (size 1.27 1.27)) hide)
+    )
     (pin "1")
     (pin "2")
@@
       (effects (font (size 1.27 1.27)) (justify left))
     )
-    (property "Footprint" "" (at 140.97 74.295 0)
+    (property "Footprint" "Capacitor_SMD:C_0603_1608Metric" (at 140.97 74.295 0)
       (effects (font (size 1.27 1.27)) hide)
     )
@@
       (effects (font (size 1.27 1.27)) hide)
     )
+    (property "MPN" "CC0603KRX7R9BB104" (at 140.97 74.295 0)
+      (effects (font (size 1.27 1.27)) hide)
+    )
     (pin "1")
     (pin "2")
@@
       (effects (font (size 1.27 1.27)) hide)
     )
+    (property "MPN" "MPU-6050" (at 140.97 99.695 0)
+      (effects (font (size 1.27 1.27)) hide)
+    )
