File: AMAS1117-1V8.kicad_sch (KiCad schematic)
At the start: 3 parts

Commit message: Add files via upload
Parts:
- C11: footprint (none) -> Capacitor_SMD:C_0603_1608Metric; MPN (none) -> CL10A106KP8NNNC
- C12: footprint (none) -> Capacitor_SMD:C_1206_3216Metric; MPN (none) -> CL31A226KPHNNNE
- U?: MPN (none) -> AMS1117-1.8
Changed lines of the file:
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@@
       (effects (font (size 1.27 1.27)) (justify left))
     )
-    (property "Footprint" "" (at 134.62 99.06 0)
+    (property "Footprint" "Capacitor_SMD:C_0603_1608Metric" (at 134.62 99.06 0)
       (effects (font (size 1.27 1.27)) hide)
     )
     (property "Datasheet" "~" (at 134.62 99.06 0)
+      (effects (font (size 1.27 1.27)) hide)
+    )
+    (property "MPN" "CL10A106KP8NNNC" (at 134.62 99.06 0)
       (effects (font (size 1.27 1.27)) hide)
     )
@@
       (effects (font (size 1.27 1.27)) (justify left))
     )
-    (property "Footprint" "" (at 163.83 99.06 0)
+    (property "Footprint" "Capacitor_SMD:C_1206_3216Metric" (at 163.83 99.06 0)
       (effects (font (size 1.27 1.27)) hide)
     )
     (property "Datasheet" "~" (at 163.83 99.06 0)
+      (effects (font (size 1.27 1.27)) hide)
+    )
+    (property "MPN" "CL31A226KPHNNNE" (at 163.83 99.06 0)
       (effects (font (size 1.27 1.27)) hide)
     )
@@
       (effects (font (size 1.27 1.27)) hide)
     )
+    (property "MPN" "AMS1117-1.8" (at 149.86 96.52 0)
+      (effects (font (size 1.27 1.27)) hide)
+    )
