File: BQ24075_charging_monitoring.kicad_sch (KiCad schematic)
At the start: 12 parts

Commit message: Add files via upload
Parts:
- removed C? (x3): 10u, symbol Device:C_Small
- removed D?: LED_RGBA, symbol Device:LED_RGBA
- removed J?: Battery_Connector, symbol Connector_Generic:Conn_01x02
- removed R? (x2): 2.2k, symbol Device:R
- removed R?: 1.78k, symbol Device:R
- removed R?: 10k, symbol Device:R
- removed R?: 20k, symbol Device:R
- removed R?: 3k, symbol Device:R
- removed U?: BQ24075RGT, Package_DFN_QFN:VQFN-16-1EP_3x3mm_P0.5mm_EP1.6x1.6mm, symbol Battery_Management:BQ24075RGT
- added C? (x3): 10uF, Capacitor_SMD:C_0603_1608Metric, symbol Device:C_Small
- added D?: LED_RGBA, LED_SMD:LED_RGB_1210, symbol Device:LED_RGBA
- added J?: Battery_Connector, Connector_PinHeader_2.54mm:PinHeader_1x02_P2.54mm_Vertical, symbol Connector_Generic:Conn_01x02
- added R?: 3k, Resistor_SMD:R_0603_1608Metric, symbol Device:R
- added R?: 20k, Resistor_SMD:R_0603_1608Metric, symbol Device:R
- added R?: 1.1k, Resistor_SMD:R_0603_1608Metric, symbol Device:R
- added R? (x2): 2.2k, Resistor_SMD:R_0603_1608Metric, symbol Device:R
- added R?: 10k, Resistor_SMD:R_0603_1608Metric, symbol Device:R
- added U?: BQ24075RGT, Package_DFN_QFN:VQFN-16-1EP_3x3mm_P0.5mm_EP1.6x1.6mm, symbol Battery_Management:BQ24075RGT
Connections:
- net +5V: now also C?.1, D?.4 (A), U?.13 (IN), U?.5 (EN2)
- net GND: now also C?.2, C?.2, C?.2, J?.2 (Pin_2), R?.2, R?.2, R?.2, R?.2, R?.2, U?.15 (SYSOFF), U?.17 (VSS), U?.4 (~{CE}), U?.6 (EN1), U?.8 (VSS)
- net bat_low_led: now also D?.3 (BK)
- net bat_voltage: now also R?.1, R?.2
- net battery+: now also C?.1, R?.1, U?.10 (OUT), U?.11 (OUT)
- net ~{chg}: now also D?.2 (GK), U?.9 (~{CHG})
- net ~{pgood}: now also D?.1 (RK), U?.7 (~{PGOOD})
- new net: R?.1, U?.12 (ILIM)
- new net: R?.1, U?.14 (TMR)
- new net: R?.1, U?.16 (ISET)
- new net: R?.1, U?.1 (TS)
- new net: C?.1, J?.1 (Pin_1), U?.2 (BAT), U?.3 (BAT)
