File: ESP32_wroom_32e.kicad_sch (KiCad schematic)
At the start: 10 parts, among them J1 Conn_01x06, SW1 SW_Push, SW2 TS-1187A-B-A-B, U1 ESP32-WROOM-32E

Commit message: Add files via upload
Parts:
- C2, C3: value 0.1u -> 0.1uF
- J1: footprint (none) -> Connector_PinHeader_2.54mm:PinHeader_1x06_P2.54mm_Vertical
- R1, R3: MPN 0603WAF1002T5E -> 0603WAF2201T5E
- R2: value 10k/5% -> 10k
- SW1: footprint TS-1187A-B-A-B:SW_TS-1187A-B-A-B -> 0000:TS-1187A-B-A-B; MPN (none) -> TS-1187A-B-A-B
- SW2: value TS-1187A-B-A-B -> RESET
Changed lines of the file:
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@@
       (effects (font (size 1.27 1.27)))
     )
-    (property "Value" "TS-1187A-B-A-B" (at 217.17 135.255 0)
+    (property "Value" "RESET" (at 217.17 135.255 0)
       (effects (font (size 1.27 1.27)))
     )
@@
       (effects (font (size 1.27 1.27)) (justify left))
     )
-    (property "Value" "0.1u" (at 230.9368 142.113 0)
+    (property "Value" "0.1uF" (at 230.9368 142.113 0)
       (effects (font (size 0.9906 0.9906)) (justify left))
     )
@@
       (effects (font (size 1.27 1.27)))
     )
-    (property "Footprint" "TS-1187A-B-A-B:SW_TS-1187A-B-A-B" (at 59.69 87.63 0)
+    (property "Footprint" "0000:TS-1187A-B-A-B" (at 59.69 87.63 0)
       (effects (font (size 1.27 1.27)) hide)
     )
     (property "Datasheet" "~" (at 59.69 87.63 0)
+      (effects (font (size 1.27 1.27)) hide)
+    )
+    (property "MPN" "TS-1187A-B-A-B" (at 59.69 92.71 0)
       (effects (font (size 1.27 1.27)) hide)
     )
@@
       (effects (font (size 1.27 1.27)) (justify left))
     )
-    (property "Value" "10k/5%" (at 230.505 131.4449 0)
+    (property "Value" "10k" (at 230.505 131.4449 0)
       (effects (font (size 1.27 1.27)) (justify left))
     )
@@
       (effects (font (size 1.27 1.27)) (justify left) hide)
     )
-    (property "Footprint" "" (at 240.665 93.98 0)
+    (property "Footprint" "Connector_PinHeader_2.54mm:PinHeader_1x06_P2.54mm_Vertical" (at 240.665 93.98 0)
       (effects (font (size 1.27 1.27)) hide)
     )
@@
       (effects (font (size 1.27 1.27)) hide)
     )
-    (property "MPN" "0603WAF1002T5E" (at 238.76 64.135 0)
+    (property "MPN" "0603WAF2201T5E" (at 238.76 64.135 0)
       (effects (font (size 1.27 1.27)) hide)
     )
@@
       (effects (font (size 1.27 1.27)) hide)
     )
-    (property "MPN" "0603WAF1002T5E" (at 227.33 64.135 0)
+    (property "MPN" "0603WAF2201T5E" (at 227.33 64.135 0)
       (effects (font (size 1.27 1.27)) hide)
     )
@@
       (effects (font (size 1.27 1.27)) (justify left))
     )
-    (property "Value" "0.1u" (at 120.015 121.92 0)
-      (effects (font (size 1.27 1.27)) (justify left))
-    )
+    (property "Value" "0.1uF" (at 120.015 121.92 0)
+      (effects (font (size 1.27 1.27)) (justify left))
+    )
