File: MAX30102.kicad_sch (KiCad schematic)
At the start: 6 parts

Commit message: Add files via upload
Parts:
- C10: footprint (none) -> Capacitor_SMD:C_1206_3216Metric; MPN (none) -> CL31A226KPHNNNE
- C7: footprint (none) -> Capacitor_SMD:C_0603_1608Metric; MPN (none) -> CL10A106KP8NNNC
- C8, C9: value 100nF -> 0.1uF; footprint (none) -> Capacitor_SMD:C_0603_1608Metric; MPN (none) -> CC0603KRX7R9BB104
- R5: value 4.7K -> 4.7k; footprint (none) -> Resistor_SMD:R_0603_1608Metric; MPN (none) -> 0603WAF4701T5E
- U?: MPN (none) -> MAX30102EFD+T
Changed lines of the file:
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@@
       (effects (font (size 1.27 1.27)) (justify left))
     )
-    (property "Value" "4.7K" (at 156.21 104.775 90)
-      (effects (font (size 1.27 1.27)) (justify left))
-    )
-    (property "Footprint" "" (at 158.115 106.68 0)
+    (property "Value" "4.7k" (at 156.21 104.775 90)
+      (effects (font (size 1.27 1.27)) (justify left))
+    )
+    (property "Footprint" "Resistor_SMD:R_0603_1608Metric" (at 158.115 106.68 0)
       (effects (font (size 1.27 1.27)) hide)
     )
@@
       (effects (font (size 1.27 1.27)) hide)
     )
+    (property "MPN" "0603WAF4701T5E" (at 158.115 106.68 0)
+      (effects (font (size 1.27 1.27)) hide)
+    )
     (pin "1")
     (pin "2")
@@
       (effects (font (size 1.27 1.27)) (justify left))
     )
-    (property "Footprint" "" (at 121.285 85.725 0)
+    (property "Footprint" "Capacitor_SMD:C_0603_1608Metric" (at 121.285 85.725 0)
       (effects (font (size 1.27 1.27)) hide)
     )
@@
       (effects (font (size 1.27 1.27)) hide)
     )
+    (property "MPN" "CL10A106KP8NNNC" (at 121.285 85.725 0)
+      (effects (font (size 1.27 1.27)) hide)
+    )
     (pin "1")
     (pin "2")
@@
       (effects (font (size 1.27 1.27)) (justify left))
     )
-    (property "Value" "100nF" (at 153.035 87.63 0)
-      (effects (font (size 1.27 1.27)) (justify left))
-    )
-    (property "Footprint" "" (at 155.575 85.725 0)
+    (property "Value" "0.1uF" (at 153.035 87.63 0)
+      (effects (font (size 1.27 1.27)) (justify left))
+    )
+    (property "Footprint" "Capacitor_SMD:C_0603_1608Metric" (at 155.575 85.725 0)
       (effects (font (size 1.27 1.27)) hide)
     )
@@
       (effects (font (size 1.27 1.27)) hide)
     )
+    (property "MPN" "CC0603KRX7R9BB104" (at 155.575 85.725 0)
+      (effects (font (size 1.27 1.27)) hide)
+    )
     (pin "1")
     (pin "2")
@@
       (effects (font (size 1.27 1.27)) (justify left))
     )
-    (property "Footprint" "" (at 160.655 85.725 0)
+    (property "Footprint" "Capacitor_SMD:C_1206_3216Metric" (at 160.655 85.725 0)
       (effects (font (size 1.27 1.27)) hide)
     )
     (property "Datasheet" "~" (at 160.655 85.725 0)
+      (effects (font (size 1.27 1.27)) hide)
+    )
+    (property "MPN" "CL31A226KPHNNNE" (at 160.655 85.725 0)
       (effects (font (size 1.27 1.27)) hide)
     )
@@
     )
     (property "Datasheet" "https://datasheets.maximintegrated.com/en/ds/MAX30102.pdf" (at 143.51 106.68 0)
+      (effects (font (size 1.27 1.27)) hide)
+    )
+    (property "MPN" "MAX30102EFD+T" (at 143.51 106.68 0)
       (effects (font (size 1.27 1.27)) hide)
     )
@@
       (effects (font (size 1.27 1.27)) (justify left))
     )
-    (property "Value" "100nF" (at 128.905 87.63 0)
-      (effects (font (size 1.27 1.27)) (justify left))
-    )
-    (property "Footprint" "" (at 126.365 85.725 0)
+    (property "Value" "0.1uF" (at 128.905 87.63 0)
+      (effects (font (size 1.27 1.27)) (justify left))
+    )
+    (property "Footprint" "Capacitor_SMD:C_0603_1608Metric" (at 126.365 85.725 0)
       (effects (font (size 1.27 1.27)) hide)
     )
@@
       (effects (font (size 1.27 1.27)) hide)
     )
+    (property "MPN" "CC0603KRX7R9BB104" (at 126.365 85.725 0)
+      (effects (font (size 1.27 1.27)) hide)
+    )
