File: V3_2A_BUCK_BOOST_MCP1700.kicad_sch (KiCad schematic)
At the start: 4 parts, among them U2 MCP1700x-330xxTT

Commit message: Add files via upload
Parts:
- C4, C6: value 10u -> 10uF; footprint (none) -> Capacitor_SMD:C_0603_1608Metric; MPN (none) -> CL10A106KP8NNNC
- C5: value 100n -> 0.1uF; footprint (none) -> Capacitor_SMD:C_0603_1608Metric; MPN (none) -> CC0603KRX7R9BB104
- U2: MPN (none) -> MCP1700T-3302E/TT
Changed lines of the file:
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@@
+      (effects (font (size 1.27 1.27)) hide)
+    )
+    (property "MPN" "MCP1700T-3302E/TT" (at 152.4 95.25 0)
       (effects (font (size 1.27 1.27)) hide)
     )
@@
       (effects (font (size 1.27 1.27)) (justify left))
     )
-    (property "Value" "100n" (at 140.97 100.965 0)
+    (property "Value" "0.1uF" (at 140.97 100.965 0)
       (effects (font (size 1.27 1.27)) (justify left))
     )
-    (property "Footprint" "" (at 139.065 99.06 0)
+    (property "Footprint" "Capacitor_SMD:C_0603_1608Metric" (at 139.065 99.06 0)
       (effects (font (size 1.27 1.27)) hide)
     )
     (property "Datasheet" "~" (at 139.065 99.06 0)
+      (effects (font (size 1.27 1.27)) hide)
+    )
+    (property "MPN" "CC0603KRX7R9BB104" (at 139.065 99.06 0)
       (effects (font (size 1.27 1.27)) hide)
     )
@@
       (effects (font (size 1.27 1.27)) (justify left))
     )
-    (property "Value" "10u" (at 128.905 100.965 0)
+    (property "Value" "10uF" (at 128.905 100.965 0)
       (effects (font (size 1.27 1.27)) (justify left))
     )
-    (property "Footprint" "" (at 127 99.06 0)
+    (property "Footprint" "Capacitor_SMD:C_0603_1608Metric" (at 127 99.06 0)
       (effects (font (size 1.27 1.27)) hide)
     )
     (property "Datasheet" "~" (at 127 99.06 0)
+      (effects (font (size 1.27 1.27)) hide)
+    )
+    (property "MPN" "CL10A106KP8NNNC" (at 127 99.06 0)
       (effects (font (size 1.27 1.27)) hide)
     )
@@
       (effects (font (size 1.27 1.27)) (justify left))
     )
-    (property "Value" "10u" (at 164.465 100.33 0)
+    (property "Value" "10uF" (at 164.465 100.33 0)
       (effects (font (size 1.27 1.27)) (justify left))
     )
-    (property "Footprint" "" (at 162.56 98.425 0)
+    (property "Footprint" "Capacitor_SMD:C_0603_1608Metric" (at 162.56 98.425 0)
       (effects (font (size 1.27 1.27)) hide)
     )
@@
       (effects (font (size 1.27 1.27)) hide)
     )
+    (property "MPN" "CL10A106KP8NNNC" (at 162.56 98.425 0)
+      (effects (font (size 1.27 1.27)) hide)
+    )
