File: haptic_motor.kicad_sch (KiCad schematic)
At the start: 1 part, among them M1 Motor_DC

Commit message: Add files via upload
Parts:
- M1: footprint (none) -> Connector_PinHeader_2.54mm:PinHeader_1x02_P2.54mm_Vertical
Changed lines of the file:
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@@
       (effects (font (size 1.27 1.27)) (justify left))
     )
-    (property "Footprint" "" (at 142.24 94.996 0)
+    (property "Footprint" "Connector_PinHeader_2.54mm:PinHeader_1x02_P2.54mm_Vertical" (at 142.24 94.996 0)
       (effects (font (size 1.27 1.27)) hide)
     )
