File: power_management.kicad_sch (KiCad schematic)
At the start: 4 parts, among them J2 USB_B_Micro, Q1 AO3401A

Commit message: Add files via upload
Parts:
- D1: footprint (none) -> Diode_SMD:D_SMA
- J2: footprint (none) -> Connector_USB:USB_Micro-B_Molex_47346-0001; MPN (none) -> 473460001
- Q1: MPN (none) -> AO3401A
- R4: footprint (none) -> Resistor_SMD:R_0603_1608Metric; MPN (none) -> 0603WAF2002T5E
Changed lines of the file:
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@@
       (effects (font (size 1.27 1.27)))
     )
-    (property "Footprint" "" (at 118.11 99.06 0)
+    (property "Footprint" "Diode_SMD:D_SMA" (at 118.11 99.06 0)
       (effects (font (size 1.27 1.27)) hide)
     )
@@
       (effects (font (size 1.27 1.27)) (justify left))
     )
-    (property "Footprint" "" (at 105.537 104.775 90)
+    (property "Footprint" "Resistor_SMD:R_0603_1608Metric" (at 105.537 104.775 90)
       (effects (font (size 1.27 1.27)) hide)
     )
     (property "Datasheet" "~" (at 107.315 104.775 0)
+      (effects (font (size 1.27 1.27)) hide)
+    )
+    (property "MPN" "0603WAF2002T5E" (at 107.315 104.775 0)
       (effects (font (size 1.27 1.27)) hide)
     )
@@
     (property "Datasheet" "http://www.aosmd.com/pdfs/datasheet/AO3401A.pdf" (at 107.315 92.71 0)
       (effects (font (size 1.27 1.27)) (justify left) hide)
+    )
+    (property "MPN" "AO3401A" (at 107.315 92.71 0)
+      (effects (font (size 1.27 1.27)) hide)
     )
     (pin "1")
@@
       (effects (font (size 1.27 1.27)))
     )
-    (property "Footprint" "" (at 113.03 47.625 0)
+    (property "Footprint" "Connector_USB:USB_Micro-B_Molex_47346-0001" (at 113.03 47.625 0)
       (effects (font (size 1.27 1.27)) hide)
     )
@@
       (effects (font (size 1.27 1.27)) hide)
     )
+    (property "MPN" "473460001" (at 109.22 46.355 0)
+      (effects (font (size 1.27 1.27)) hide)
+    )
